File: hardware/designs/mcu-modulino/led-matrix.kicad_sch (KiCad schematic)
At the start: 96 parts

Commit message: chore: title schematics
Other:
- title: (none) -> Charlieplexed LED Matrix
Changed lines of the file:
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@@
 	(generator_version "10.0")
 	(paper "A4")
+	(title_block
+		(title "Charlieplexed LED Matrix")
+		(rev "A")
+	)
 	(rectangle
 		(start 235.712 132.842)
