File: hardware/designs/mcu-modulino/usb-uart.kicad_sch (KiCad schematic)
At the start: 19 parts, among them J1 USB_C_Receptacle_USB2.0_14P, J2 FTDI Header, J3 Modem, U1 CP2102N-Axx-xQFN28

Commit message: chore: title schematics
Other:
- title: (none) -> USB-to-UART Bridge Controller
Changed lines of the file:
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@@
 	(generator_version "10.0")
 	(paper "A4")
+	(title_block
+		(title "USB-to-UART Bridge Controller")
+		(rev "B")
+	)
 	(rectangle
 		(start 75.6106 78.9275)
