File: hardware/designs/mcu-modulino/mcu-modulino.kicad_sch (KiCad schematic)
At the start: 52 parts, among them J4 PROG, J5 JTAG, J6 Stemma QT, Q1 BC847BDW1, SW1 RESET, SW2 BOOT, U2 NCP1117-3.3_SOT223, U3 ESP32-WROVER-E, U4 IS31FL3731-QF, X1 EYESPI, X2 EYESPI, X3 EYESPI

Commit message: feat: remove charlieplex matrix from board rev c
Parts:
- added R15, R16: 4.7k, Resistor_SMD:R_0603_1608Metric_Pad0.98x0.95mm_HandSolder, symbol Device:R_US
- C17, C18: now in the parts list
Connections:
- net +3.3V: now also X3.10, R15.1, R16.1; no longer X3.16
- net GND: now also X3.16; no longer X3.10
- net HSPI_CS: now also RN1.1, U3.23 (MTDO)
- net RF_RST: now also U3.25 (GPIO0)
- net SCL: now also R15.2
- net SDA: now also R16.2
- net TFT_RST: now also U3.24 (GPIO2)
- net VSPI_CS: now also RN1.2, U3.29 (IO5)
- net LED Matrix/CB4: now reaches U4.10 (CB4)
- net LED Matrix/CB5: now reaches U4.11 (CB5)
- net LED Matrix/CB6: now reaches U4.12 (CB6)
- net LED Matrix/CB7: now reaches U4.13 (CB7)
- net LED Matrix/CB8: now reaches U4.14 (CB8)
- no-connect marks 20 -> 13
Other:
- sheet LED Matrix ports: added CB4, CB5, CB6, CB7, CB8; removed none
- title: (none) -> Microcontroller Modulino
- moved on the sheet: C17, C18, RN1A, RN1B
