File: hardware/designs/mcu-module/mcu-module.kicad_sch (KiCad schematic)
At the start: 54 parts, among them J4 PROG, J5 JTAG, J6 Stemma QT, Q1 BC847BDW1, SW1 RESET, SW2 BOOT, U2 NCP1117-3.3_SOT223, U3 ESP32-WROVER-E, U4 IS31FL3731-QF, X1 EYESPI, X2 EYESPI, X3 EYESPI

Commit message: rename: -modulino boards to -module (trademark)
"Modulino" is Arduino's own trademark (Modulino®/™), used across their Plug and Make Kit product line.

Renaming this project's board naming convention away from it to avoid the conflict: mcu-modulino -> mcu-module, modulino-template -> module-template, radio-modulino -> radio-module.

Also collapses the stale mcu-modulino-REV-C internal KiCad instance-path label down to the flat mcu-module name, since revision tracking belongs to git and KiCad's own ${REVISION} title block variable, not a name baked into the project files.
Other:
- title: Microcontroller Modulino -> Microcontroller Module
